File: schematics/controller layout.sch (KiCad schematic (older format))
At the start: 12 parts, among them J1 Conn_01x12, J2 Conn_01x16, SW1 SW_SPDT_MSM, SW1 SW_SPST, SW2 SW_SPDT_MSM, SW3 SW_SPDT_MSM, SW4 SW_SPST

Commit message: Update schematics
Parts:
- removed BT1: LiPo single cell, symbol Device:Battery_Cell
- removed J1: Conn_01x12, symbol Connector_Generic:Conn_01x12
- removed J2: Conn_01x16, symbol Connector_Generic:Conn_01x16
- removed SW1: SW_SPST, symbol Switch:SW_SPST
- added SW5: (no value), symbol Switch:SW_SPDT
Connections:
- net D5: now also SW5.1 (A)
- net GND: now also SW5.2 (B)
Other:
- note added: "Versioning:\nv1.0 - original\nv1.1 - moved SW2 to different XBee3 pins\nv2.0 - range extender is now part of the controller"
- note removed: "Range Extender"
- note removed: "Versioning:\nv1.0 - original\nv1.1 - moved SW2 to different XBee3 pins"
- moved on the sheet: BT1, J1, J2, RV1, SW1, SW2, SW3, SW4
