File: schematics/winch box.sch (KiCad schematic (older format))
At the start: 6 parts, among them J1 ISD04 motor controller, J2 AD-02BFFB-QL8AP0, J3 AD-02PMMS-QC8001, U1 tic-t249

Commit message: Update schematics
Parts:
- removed J1: ISD04 motor controller, symbol Connector_Generic:Conn_01x06
- removed PS1: VTX-214-015-124, Converter_ACDC:Converter_ACDC_Vigortronix_VTX-214-015-1xx_THT, symbol Converter_ACDC:VTX-214-015-124
- added BT1: Hikoki MultiVolt 36V, symbol Device:Battery
- added J3: Molex 43645-0400, symbol Connector:Conn_01x04_Female
- added J4: Molex 43640-0401, symbol Connector:Conn_01x04_Male
- added M1: 23HS30-2804S-PG4, symbol Motor:Stepper_Motor_bipolar
- renumbered J2 to J1, J3 to J2
Connections:
- net GND is gone; now on net A+: J1.3 (Pin_3), JP4.2 (Pin_2), U1.10 (GND), U1.16 (GND)
- net V+ is gone; now on net 5V: J1.1 (Pin_1), U1.15 (VIN)
- net 5V: now also U1.20 (B2), J3.4 (Pin_4), J4.4 (Pin_4), M1.3
- net DOUT: now also U1.17 (A1), J3.2 (Pin_2)
- net at J2.1 (Pin_1): now also BT1.1 (+)
- net at J2.3 (Pin_3): now also BT1.2 (-)
- net A+: now reaches U1.18 (A2)
- net A+: now also J3.1 (Pin_1), J4.1 (Pin_1), M1.1
- net B-: now reaches U1.19 (B1)
- net B-: now also J3.3 (Pin_3), J4.3 (Pin_3), M1.4
- net DIR: no longer names the net of U1.12 (DIR)
- net STEP: no longer names the net of U1.11 (STEP)
- new net A-: J4.2 (Pin_2), M1.2 (-)
Other:
- moved on the sheet: J1, J2, JP4, U1
